File: Project/Project.sch (KiCad schematic (older format))
At the start: 46 parts, among them J1 Conn_01x05_Male, J2 USB_OTG, J3 Conn_01x09_Male, J4 Conn_01x03_Female, J5 Conn_Coaxial, SW1 SW_Push, SW2 SW_Push, SW3 SW_Push, U1 CMWX1ZZABZ-078, U2 LM1117ADJ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

Commit message: all routes done and copperlayer
Parts:
- U1: footprint RF_Module:CMWX1ZZABZ -> lab1_CMWX1ZZABZ-078:CMWX1ZZABZ_longer_pads
Connections:
- net 1pps(1_pulse_per_second): now also U1.18 (PA10/USART1_RX); no longer U1.24 (PA2/ADC2)
- net TX: now also U1.22 (PA4/ADC4/DAC1); no longer U1.18 (PA10/USART1_RX)
- net temperature: now also U1.21 (PA5/ADC5/DAC2); no longer U1.22 (PA4/ADC4/DAC1)
- net at R1.2: now also U1.24 (PA2/ADC2); no longer U1.21 (PA5/ADC5/DAC2)
Changed lines of the file:
@@
 3DF(3D-FiX_indicator)
-Wire Wire Line
-	2950 3050 3350 3050
 Wire Wire Line
 	3150 3150 3350 3150
 Text Label 4900 6800 0    50   ~ 0
 temperature
-Text Label 2850 3250 2    50   ~ 0
+Text Label 3350 3350 2    50   ~ 0
 temperature
 Wire Wire Line
@@
 F 0 "U1" H 4250 2261 50  0000 C CNN
 F 1 "CMWX1ZZABZ-078" H 4250 2170 50  0000 C CNN
-F 2 "RF_Module:CMWX1ZZABZ" H 4250 3850 50  0001 C CNN
+F 2 "lab1_CMWX1ZZABZ-078:CMWX1ZZABZ_longer_pads" H 4250 3850 50  0001 C CNN
 F 3 "https://wireless.murata.com/RFM/data/type_abz.pdf" H 6700 2350 50  0001 C CNN
 	1    4250 3850
@@
 Wire Wire Line
 	1350 2500 1350 2750
-Text Label 2750 3650 0    50   ~ 0
+Text Label 2850 3250 0    50   ~ 0
 TX
 Text Label 2700 3450 0    50   ~ 0
@@
 Wire Wire Line
 	9250 2900 9650 2900
-Text Label 2950 3050 2    50   ~ 0
+Text Label 2750 3650 2    50   ~ 0
 1pps(1_pulse_per_second)
 $Comp
@@
 	1550 3350 1550 3200
 Wire Wire Line
-	1550 3350 3350 3350
-Wire Wire Line
 	1550 2500 1550 2900
 NoConn ~ 1450 2800
@@
 Wire Wire Line
 	10200 2200 10400 2200
+Wire Wire Line
+	1550 3350 2050 3350
+Wire Wire Line
+	2050 3350 2050 3050
+Wire Wire Line
+	2050 3050 3350 3050
 $EndSCHEMATC

Commit message: changed some fottprints that where wrong
Parts:
- J3: footprint Connector_PinHeader_2.54mm:PinHeader_1x09_P2.54mm_Horizontal -> Connector_PinHeader_2.54mm:PinHeader_1x09_P2.54mm_Vertical
Changed lines of the file:
@@
 F 0 "J3" V 1085 2278 50  0000 C CNN
 F 1 "Conn_01x09_Male" V 1176 2278 50  0000 C CNN
-F 2 "Connector_PinHeader_2.54mm:PinHeader_1x09_P2.54mm_Horizontal" H 1250 2300 50  0001 C CNN
+F 2 "Connector_PinHeader_2.54mm:PinHeader_1x09_P2.54mm_Vertical" H 1250 2300 50  0001 C CNN
 F 3 "~" H 1250 2300 50  0001 C CNN
 	1    1250 2300

Commit message: updated schematic
Parts:
- removed R3: 330, Resistor_SMD:R_0805_2012Metric_Pad1.15x1.40mm_HandSolder, symbol Device:R
- removed R4: 560, Resistor_SMD:R_0805_2012Metric_Pad1.15x1.40mm_HandSolder, symbol Device:R
- removed U2: LM1117ADJ, Package_TO_SOT_SMD:SOT-223, symbol LM117ADJ:LM1117ADJ
- added C23: 10n, Capacitor_SMD:C_0805_2012Metric_Pad1.15x1.40mm_HandSolder, symbol Device:C
- added U2: SPX3819M5-L-3-3, Package_TO_SOT_SMD:SOT-23-5, symbol Regulator_Linear:SPX3819M5-L-3-3
Connections:
- net +3V3: now also C11.2, C12.2, U2.5 (OUT); no longer C11.1, C12.1
- net GND: now also C11.1, C12.1, C23.1, U2.2 (GND); no longer C11.2, C12.2
- net at C10.1, C13.1, C15.1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: now also U2.1 (IN), U2.3 (EN)
- new net: C23.2, U2.4 (BP)
Other:
- moved on the sheet: C10, C11, C12, C13, C14, C15, C9

Commit message: final design probably
Parts:
- C18: value 4.7u -> 0.1u
- C3, C5: value 100n -> 10u
- C4: value 100n -> 0.1n
- C6, C8: value 100n -> 1u
- C7: value 100n -> 0.1
Changed lines of the file:
@@
 P 3950 2000
 F 0 "C6" H 4065 2046 50  0000 L CNN
-F 1 "100n" H 4065 1955 50  0000 L CNN
+F 1 "1u" H 4065 1955 50  0000 L CNN
 F 2 "Capacitor_SMD:C_0805_2012Metric_Pad1.15x1.40mm_HandSolder" H 3988 1850 50  0001 C CNN
 F 3 "~" H 3950 2000 50  0001 C CNN
@@
 P 3950 2200
 F 0 "C7" H 4065 2246 50  0000 L CNN
-F 1 "100n" H 4065 2155 50  0000 L CNN
+F 1 "0.1" H 4065 2155 50  0000 L CNN
 F 2 "Capacitor_SMD:C_0805_2012Metric_Pad1.15x1.40mm_HandSolder" H 3988 2050 50  0001 C CNN
 F 3 "~" H 3950 2200 50  0001 C CNN
@@
 P 3950 1800
 F 0 "C5" V 3698 1800 50  0000 C CNN
-F 1 "100n" V 3789 1800 50  0000 C CNN
+F 1 "10u" V 3789 1800 50  0000 C CNN
 F 2 "Capacitor_SMD:C_0805_2012Metric_Pad1.15x1.40mm_HandSolder" H 3988 1650 50  0001 C CNN
 F 3 "~" H 3950 1800 50  0001 C CNN
@@
 P 3300 2000
 F 0 "C3" H 3415 2046 50  0000 L CNN
-F 1 "100n" H 3415 1955 50  0000 L CNN
+F 1 "10u" H 3415 1955 50  0000 L CNN
 F 2 "Capacitor_SMD:C_0805_2012Metric_Pad1.15x1.40mm_HandSolder" H 3338 1850 50  0001 C CNN
 F 3 "~" H 3300 2000 50  0001 C CNN
@@
 P 3300 2200
 F 0 "C4" H 3415 2246 50  0000 L CNN
-F 1 "100n" H 3415 2155 50  0000 L CNN
+F 1 "0.1n" H 3415 2155 50  0000 L CNN
 F 2 "Capacitor_SMD:C_0805_2012Metric_Pad1.15x1.40mm_HandSolder" H 3338 2050 50  0001 C CNN
 F 3 "~" H 3300 2200 50  0001 C CNN
@@
 P 4400 1850
 F 0 "C8" H 4515 1896 50  0000 L CNN
-F 1 "100n" H 4515 1805 50  0000 L CNN
+F 1 "1u" H 4515 1805 50  0000 L CNN
 F 2 "Capacitor_SMD:C_0805_2012Metric_Pad1.15x1.40mm_HandSolder" H 4438 1700 50  0001 C CNN
 F 3 "~" H 4400 1850 50  0001 C CNN
@@
 U 1 1 5E43DB6D
 P 9700 1650
-F 0 "C17" H 9815 1696 50  0000 L CNN
-F 1 "4.7u" H 9815 1605 50  0000 L CNN
+F 0 "C17" H 9550 1550 50  0000 L CNN
+F 1 "4.7u" H 9750 1550 50  0000 L CNN
 F 2 "Capacitor_SMD:C_0805_2012Metric_Pad1.15x1.40mm_HandSolder" H 9738 1500 50  0001 C CNN
 F 3 "~" H 9700 1650 50  0001 C CNN
@@
 P 3450 6250
 F 0 "C18" H 3565 6296 50  0000 L CNN
-F 1 "4.7u" H 3565 6205 50  0000 L CNN
+F 1 "0.1u" H 3565 6205 50  0000 L CNN
 F 2 "Capacitor_SMD:C_0805_2012Metric_Pad1.15x1.40mm_HandSolder" H 3488 6100 50  0001 C CNN
 F 3 "~" H 3450 6250 50  0001 C CNN
@@
 U 1 1 5E3FBD78
 P 9200 2350
-F 0 "C16" H 9315 2396 50  0000 L CNN
-F 1 "4.7u" H 9315 2305 50  0000 L CNN
+F 0 "C16" H 9200 2250 50  0000 L CNN
+F 1 "4.7u" H 9050 2250 50  0000 L CNN
 F 2 "Capacitor_SMD:C_0805_2012Metric_Pad1.15x1.40mm_HandSolder" H 9238 2200 50  0001 C CNN
 F 3 "~" H 9200 2350 50  0001 C CNN
@@
 U 1 1 5E403B6F
 P 9400 2200
-F 0 "D2" H 9393 2416 50  0000 C CNN
+F 0 "D2" H 9400 2100 50  0000 C CNN
 F 1 "LED" H 9393 2325 50  0000 C CNN
 F 2 "LED_SMD:LED_0805_2012Metric_Pad1.15x1.40mm_HandSolder" H 9400 2200 50  0001 C CNN

Commit message: gerber
Parts:
- C21: value 100n -> 100p
- C4: value 0.1n -> 0.1u
- C7: value 0.1 -> 0.1u
Changed lines of the file:
@@
 P 3950 2200
 F 0 "C7" H 4065 2246 50  0000 L CNN
-F 1 "0.1" H 4065 2155 50  0000 L CNN
+F 1 "0.1u" H 4065 2155 50  0000 L CNN
 F 2 "Capacitor_SMD:C_0805_2012Metric_Pad1.15x1.40mm_HandSolder" H 3988 2050 50  0001 C CNN
 F 3 "~" H 3950 2200 50  0001 C CNN
@@
 P 3300 2200
 F 0 "C4" H 3415 2246 50  0000 L CNN
-F 1 "0.1n" H 3415 2155 50  0000 L CNN
+F 1 "0.1u" H 3415 2155 50  0000 L CNN
 F 2 "Capacitor_SMD:C_0805_2012Metric_Pad1.15x1.40mm_HandSolder" H 3338 2050 50  0001 C CNN
 F 3 "~" H 3300 2200 50  0001 C CNN
@@
 P 5500 5200
 F 0 "C21" V 5248 5200 50  0000 C CNN
-F 1 "100n" V 5650 5200 50  0000 C CNN
+F 1 "100p" V 5650 5200 50  0000 C CNN
 F 2 "Capacitor_SMD:C_0805_2012Metric_Pad1.15x1.40mm_HandSolder" H 5538 5050 50  0001 C CNN
 F 3 "~" H 5500 5200 50  0001 C CNN

Commit message: final design
Connections:
- net +3V3: no longer J3.1 (Pin_1)
- net VbAt: no longer names the net of J3.3 (Pin_3)
Changed lines of the file:
@@
 	0    1    1    0
 $EndComp
-$Comp
-L power:+3.3V #PWR0110
-U 1 1 5E50E564
-P 1650 2700
-F 0 "#PWR0110" H 1650 2550 50  0001 C CNN
-F 1 "+3.3V" H 1665 2873 50  0000 C CNN
-F 2 "" H 1650 2700 50  0001 C CNN
-F 3 "" H 1650 2700 50  0001 C CNN
-	1    1650 2700
-	-1   0    0    1
-$EndComp
-Wire Wire Line
-	1650 2500 1650 2700
 Text Label 1550 2750 1    50   ~ 0
 enable
-Text Label 1450 2800 1    50   ~ 0
-VbAt
-Wire Wire Line
-	1450 2500 1450 2800
 Wire Wire Line
 	1350 2500 1350 2750
@@
 Wire Wire Line
 	1550 2500 1550 2900
-NoConn ~ 1450 2800
 NoConn ~ 1450 2500
 Wire Wire Line
@@
 Wire Wire Line
 	7400 4250 7400 3400
+NoConn ~ 1650 2500
 $EndSCHEMATC
