File: Project/Project.kicad_pcb (KiCad board)
At the start: 2 copper layers, 45 parts, among them J1 Conn_01x05_Male, J2 USB_OTG, J3 Conn_01x09_Male, J4 Conn_01x03_Female, J5 Conn_Coaxial, SW1 SW_Push, SW2 SW_Push, SW3 SW_Push, U1 CMWX1ZZABZ-078, U2 SPX3819M5-L-3-3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

Commit message: done
Parts:
- C21: value 100n -> 100p
- C4: value 0.1n -> 0.1u
- C7: value 0.1 -> 0.1u
Changed lines of the file:
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@@
       (drillshape 0)
       (scaleselection 1)
-      (outputdirectory "./"))
+      (outputdirectory "gerber/"))
   )
   (net 0 "")
@@
       (effects (font (size 1 1) (thickness 0.15)))
     )
-    (fp_text value 0.1n (at 0 1.65) (layer F.Fab)
+    (fp_text value 0.1u (at 0 1.65) (layer F.Fab)
       (effects (font (size 1 1) (thickness 0.15)))
     )
@@
       (effects (font (size 1 1) (thickness 0.15)))
     )
-    (fp_text value 0.1 (at 0 1.65) (layer F.Fab)
+    (fp_text value 0.1u (at 0 1.65) (layer F.Fab)
       (effects (font (size 1 1) (thickness 0.15)))
     )
@@
       (effects (font (size 1 1) (thickness 0.15)))
     )
-    (fp_text value 100n (at 0 1.65 270) (layer F.Fab)
+    (fp_text value 100p (at 0 1.65 270) (layer F.Fab)
       (effects (font (size 1 1) (thickness 0.15)))
     )
@@
     (connect_pads (clearance 0.508))
     (min_thickness 0.254)
-    (fill (arc_segments 32) (thermal_gap 0.508) (thermal_bridge_width 0.508))
+    (fill yes (arc_segments 32) (thermal_gap 0.508) (thermal_bridge_width 0.508))
     (polygon
       (pts
@@
     (connect_pads (clearance 0.508))
     (min_thickness 0.254)
-    (fill (arc_segments 32) (thermal_gap 0.508) (thermal_bridge_width 0.508))
+    (fill yes (arc_segments 32) (thermal_gap 0.508) (thermal_bridge_width 0.508))
     (polygon
       (pts

Commit message: final design
Connections:
- J3 pad 1: +3V3 -> Net-(J3-Pad1)
Routing:
- net +3V3: track 193.2 -> 249.3 mm, vias 4 -> 5
- net GND: track 19.3 -> 40.0 mm, vias 5 -> 10
- net /NRST: track 22.5 -> 36.9 mm, vias 1 -> 2
- net Net-(R7-Pad1): track 17.4 -> 27.1 mm
- net Net-(R6-Pad1): track 20.5 -> 30.2 mm
- net Net-(C10-Pad1): track 83.9 -> 87.0 mm
- net Net-(R5-Pad2): track 5.80 -> 7.60 mm
- net Net-(R1-Pad2): track 3.97 -> 5.77 mm
- net /temperature: track 17.8 -> 19.6 mm
- net /TX: track 22.6 -> 24.4 mm
- net /SWDIO: track 21.8 -> 23.6 mm
- net /SWCLK: track 24.4 -> 26.2 mm
- net /RX: track 22.1 -> 23.9 mm
- net /3DF(3D-FiX_indicator): track 21.1 -> 22.9 mm
- net /1pps(1_pulse_per_second): track 29.8 -> 31.6 mm
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
Commit message: final design
Routing:
- net Net-(U1-Pad30): track 0.00 -> 1.80 mm
- net Net-(U1-Pad9): track 0.00 -> 1.80 mm
- net Net-(U1-Pad8): track 0.00 -> 1.80 mm
- net Net-(U1-Pad47): track 0.00 -> 1.80 mm
- net Net-(U1-Pad46): track 0.00 -> 1.80 mm
- net Net-(U1-Pad45): track 0.00 -> 1.80 mm
- net Net-(U1-Pad38): track 0.00 -> 1.80 mm
- net Net-(U1-Pad36): track 0.00 -> 1.80 mm
- net Net-(U1-Pad35): track 0.00 -> 1.80 mm
- net Net-(U1-Pad33): track 0.00 -> 1.80 mm
- net Net-(U1-Pad31): track 0.00 -> 1.80 mm
- net Net-(U1-Pad29): track 0.00 -> 1.80 mm
- net Net-(U1-Pad28): track 0.00 -> 1.80 mm
- net Net-(U1-Pad20): track 0.00 -> 1.80 mm
- net Net-(U1-Pad2): track 0.00 -> 1.80 mm
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Changed lines of the file:
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@@
     (thickness 1.6)
     (drawings 6)
-    (tracks 311)
+    (tracks 337)
     (zones 0)
     (modules 45)
@@
   (segment (start 283.356 275.952) (end 282.082 275.952) (width 0.25) (layer F.Cu) (net 7))
   (segment (start 283.718 275.59) (end 283.356 275.952) (width 0.25) (layer F.Cu) (net 7))
+  (segment (start 282.082 275.952) (end 280.282 275.952) (width 0.25) (layer F.Cu) (net 7))
+  (segment (start 282.082 279.952) (end 280.282 279.952) (width 0.25) (layer F.Cu) (net 8))
+  (segment (start 269.882 277.552) (end 268.082 277.552) (width 0.25) (layer F.Cu) (net 9))
+  (segment (start 269.882 275.152) (end 268.082 275.152) (width 0.25) (layer F.Cu) (net 10))
+  (segment (start 269.882 274.352) (end 268.092 274.352) (width 0.25) (layer F.Cu) (net 11))
+  (segment (start 269.882 273.552) (end 268.092 273.552) (width 0.25) (layer F.Cu) (net 12))
+  (segment (start 269.882 272.752) (end 268.092 272.752) (width 0.25) (layer F.Cu) (net 13))
+  (segment (start 269.882 271.952) (end 268.092 271.952) (width 0.25) (layer F.Cu) (net 14))
+  (segment (start 270.682 268.902) (end 270.682 270.702) (width 0.25) (layer F.Cu) (net 15))
+  (segment (start 279.482 282.002) (end 279.482 283.802) (width 0.25) (layer F.Cu) (net 16))
+  (segment (start 278.682 282.002) (end 278.682 283.802) (width 0.25) (layer F.Cu) (net 17))
+  (segment (start 277.082 282.002) (end 277.082 283.802) (width 0.25) (layer F.Cu) (net 18))
+  (segment (start 275.482 282.002) (end 275.482 283.802) (width 0.25) (layer F.Cu) (net 19))
+  (segment (start 274.682 283.792) (end 274.692 283.802) (width 0.25) (layer F.Cu) (net 20))
+  (segment (start 274.682 282.002) (end 274.682 283.792) (width 0.25) (layer F.Cu) (net 20))
+  (segment (start 273.882 282.002) (end 273.882 283.802) (width 0.25) (layer F.Cu) (net 21))
+  (segment (start 273.082 282.002) (end 273.082 283.802) (width 0.25) (layer F.Cu) (net 22))
+  (segment (start 271.482 268.902) (end 271.482 270.702) (width 0.25) (layer F.Cu) (net 23))
+  (segment (start 272.282 268.902) (end 272.282 270.702) (width 0.25) (layer F.Cu) (net 24))
+  (segment (start 273.082 268.902) (end 273.082 270.702) (width 0.25) (layer F.Cu) (net 25))
+  (segment (start 273.882 268.902) (end 273.882 270.702) (width 0.25) (layer F.Cu) (net 26))
+  (segment (start 278.682 268.902) (end 278.682 270.702) (width 0.25) (layer F.Cu) (net 27))
+  (segment (start 279.482 268.902) (end 279.482 270.702) (width 0.25) (layer F.Cu) (net 28))
+  (segment (start 282.082 272.752) (end 280.282 272.752) (width 0.25) (layer F.Cu) (net 29))
   (via (at 255.82 247.63) (size 0.8) (drill 0.3) (layers F.Cu B.Cu) (net 30))
   (segment (start 272.282 281.102) (end 272.3 281.084) (width 0.5) (layer F.Cu) (net 30))
@@
   (segment (start 266.820975 277.501025) (end 267.67195 278.352) (width 0.2) (layer F.Cu) (net 50))
   (segment (start 268.082 278.352) (end 269.882 278.352) (width 0.25) (layer F.Cu) (net 50))
+  (segment (start 282.082 274.352) (end 280.282 274.352) (width 0.25) (layer F.Cu) (net 51))
+  (segment (start 282.082 273.552) (end 280.282 273.552) (width 0.25) (layer F.Cu) (net 52))
   (segment (start 297.532 254.448) (end 297.212 254.128) (width 0.5) (layer F.Cu) (net 53))
   (segment (start 297.532 256.838) (end 297.532 254.448) (width 0.5) (layer F.Cu) (net 53))
